Commit message: added env and different drone colors

File: src/drone_swarm/urdf/parts/base_link.urdf.xacro (robot description, xacro)
@@ -11,5 +11,10 @@
       <origin xyz="0 0 0" rpy="0 0 0"/>
       <geometry><box size="${body_x} ${body_y} ${body_z}"/></geometry>
-      <material name="dark_grey"/>
+      <xacro:if value="${ns == 'evader'}">
+        <material name="ev_black"/>
+      </xacro:if>
+      <xacro:unless value="${ns == 'evader'}">
+        <material name="dark_grey"/>
+      </xacro:unless>
     </visual>
     <collision>
@@ -21,20 +26,24 @@
       <origin xyz=" ${arm_len/2+body_x/4} 0 0"/>
       <geometry><box size="${arm_len/2} ${arm_w} ${arm_w}"/></geometry>
-      <material name="grey"/>
+      <xacro:if value="${ns == 'evader'}"><material name="ev_white"/></xacro:if>
+      <xacro:unless value="${ns == 'evader'}"><material name="grey"/></xacro:unless>
     </visual>
     <visual>
       <origin xyz="-${arm_len/2+body_x/4} 0 0"/>
       <geometry><box size="${arm_len/2} ${arm_w} ${arm_w}"/></geometry>
-      <material name="grey"/>
+      <xacro:if value="${ns == 'evader'}"><material name="ev_white"/></xacro:if>
+      <xacro:unless value="${ns == 'evader'}"><material name="grey"/></xacro:unless>
     </visual>
     <visual>
       <origin xyz="0  ${arm_len/2+body_y/4} 0"/>
       <geometry><box size="${arm_w} ${arm_len/2} ${arm_w}"/></geometry>
-      <material name="grey"/>
+      <xacro:if value="${ns == 'evader'}"><material name="ev_white"/></xacro:if>
+      <xacro:unless value="${ns == 'evader'}"><material name="grey"/></xacro:unless>
     </visual>
     <visual>
       <origin xyz="0 -${arm_len/2+body_y/4} 0"/>
       <geometry><box size="${arm_w} ${arm_len/2} ${arm_w}"/></geometry>
-      <material name="grey"/>
+      <xacro:if value="${ns == 'evader'}"><material name="ev_white"/></xacro:if>
+      <xacro:unless value="${ns == 'evader'}"><material name="grey"/></xacro:unless>
     </visual>
     <!-- ── motor mounts at arm tips (visual only) ── -->
@@ -42,22 +51,31 @@
       <origin xyz=" ${arm_len} 0          ${mount_z}"/>
       <geometry><cylinder radius="${mount_r}" length="${mount_h}"/></geometry>
-      <material name="dark_grey"/>
+      <xacro:if value="${ns == 'evader'}"><material name="ev_black"/></xacro:if>
+      <xacro:unless value="${ns == 'evader'}"><material name="dark_grey"/></xacro:unless>
     </visual>
     <visual>
       <origin xyz="-${arm_len} 0          ${mount_z}"/>
       <geometry><cylinder radius="${mount_r}" length="${mount_h}"/></geometry>
-      <material name="dark_grey"/>
+      <xacro:if value="${ns == 'evader'}"><material name="ev_black"/></xacro:if>
+      <xacro:unless value="${ns == 'evader'}"><material name="dark_grey"/></xacro:unless>
     </visual>
     <visual>
       <origin xyz="0           ${arm_len} ${mount_z}"/>
       <geometry><cylinder radius="${mount_r}" length="${mount_h}"/></geometry>
-      <material name="dark_grey"/>
+      <xacro:if value="${ns == 'evader'}"><material name="ev_black"/></xacro:if>
+      <xacro:unless value="${ns == 'evader'}"><material name="dark_grey"/></xacro:unless>
     </visual>
     <visual>
       <origin xyz="0          -${arm_len} ${mount_z}"/>
       <geometry><cylinder radius="${mount_r}" length="${mount_h}"/></geometry>
-      <material name="dark_grey"/>
+      <xacro:if value="${ns == 'evader'}"><material name="ev_black"/></xacro:if>
+      <xacro:unless value="${ns == 'evader'}"><material name="dark_grey"/></xacro:unless>
     </visual>
   </link>
-  <gazebo reference="base_link"><material>Gazebo/DarkGrey</material></gazebo>
+  <xacro:if value="${ns == 'evader'}">
+    <gazebo reference="base_link"><material>Gazebo/Black</material></gazebo>
+  </xacro:if>
+  <xacro:unless value="${ns == 'evader'}">
+    <gazebo reference="base_link"><material>Gazebo/DarkGrey</material></gazebo>
+  </xacro:unless>
 </robot>

File: src/drone_swarm/urdf/parts/materials.urdf.xacro (robot description, xacro)
@@ -6,3 +6,7 @@
   <material name="red">      <color rgba="0.85 0.10 0.10 0.85"/></material>
   <material name="blue">     <color rgba="0.10 0.25 0.85 0.85"/></material>
+  <!-- Evader-specific palette: body=black, arms=white, rotors=green -->
+  <material name="ev_black">  <color rgba="0.05 0.05 0.05 1.00"/></material>
+  <material name="ev_white">  <color rgba="0.95 0.95 0.95 1.00"/></material>
+  <material name="ev_green">  <color rgba="0.10 0.80 0.10 1.00"/></material>
 </robot>

File: src/drone_swarm/urdf/quadrotor.urdf.xacro (robot description, xacro)
@@ -16,9 +16,17 @@
   <xacro:include filename="parts/rotor.urdf.xacro"/>
   <xacro:include filename="parts/gazebo_plugins.urdf.xacro"/>
-  <!-- 4 rotors: front/rear CW (red), left/right CCW (blue) -->
-  <xacro:rotor name="rotor_front" px=" ${arm_len}" py=" 0"          rviz_mat="red"  gz_mat="Red"/>
-  <xacro:rotor name="rotor_rear"  px="-${arm_len}" py=" 0"          rviz_mat="red"  gz_mat="Red"/>
-  <xacro:rotor name="rotor_left"  px=" 0"          py=" ${arm_len}" rviz_mat="blue" gz_mat="Blue"/>
-  <xacro:rotor name="rotor_right" px=" 0"          py="-${arm_len}" rviz_mat="blue" gz_mat="Blue"/>
+  <!-- 4 rotors: formation drones = red/blue; evader = all green -->
+  <xacro:if value="${ns == 'evader'}">
+    <xacro:rotor name="rotor_front" px=" ${arm_len}" py=" 0"          rviz_mat="ev_green" gz_mat="Green"/>
+    <xacro:rotor name="rotor_rear"  px="-${arm_len}" py=" 0"          rviz_mat="ev_green" gz_mat="Green"/>
+    <xacro:rotor name="rotor_left"  px=" 0"          py=" ${arm_len}" rviz_mat="ev_green" gz_mat="Green"/>
+    <xacro:rotor name="rotor_right" px=" 0"          py="-${arm_len}" rviz_mat="ev_green" gz_mat="Green"/>
+  </xacro:if>
+  <xacro:unless value="${ns == 'evader'}">
+    <xacro:rotor name="rotor_front" px=" ${arm_len}" py=" 0"          rviz_mat="red"  gz_mat="Red"/>
+    <xacro:rotor name="rotor_rear"  px="-${arm_len}" py=" 0"          rviz_mat="red"  gz_mat="Red"/>
+    <xacro:rotor name="rotor_left"  px=" 0"          py=" ${arm_len}" rviz_mat="blue" gz_mat="Blue"/>
+    <xacro:rotor name="rotor_right" px=" 0"          py="-${arm_len}" rviz_mat="blue" gz_mat="Blue"/>
+  </xacro:unless>
   <!-- Gazebo plugins (force input + odometry output) -->
   <xacro:gazebo_plugins ns="${ns}"/>
